File: pcb/pcb.kicad_sch (KiCad schematic)
At the start: 1 part, among them U1 ATmega32-16P

Commit message: actualizo circuito
Parts:
- added C1: C_Polarized, symbol Device:C_Polarized
- added D1: LED, symbol Device:LED
- added J1: encoder, Connector_PinSocket_2.54mm:PinSocket_1x05_P2.54mm_Vertical, symbol Connector_Generic:Conn_01x05
- added J2: programmer, Connector_PinHeader_2.54mm:PinHeader_1x04_P2.54mm_Vertical, symbol Connector_Generic:Conn_01x04
- added J3: oled display, Connector_PinHeader_2.54mm:PinHeader_1x20_P2.54mm_Vertical, symbol Connector_Generic:Conn_01x20
- added J4: usb-ttl, Connector_PinHeader_2.54mm:PinHeader_1x04_P2.54mm_Vertical, symbol Connector_Generic:Conn_01x04
- added R1, R2: R_US, symbol Device:R_US
Connections:
- net +5V: now reaches U1.10 (VCC)
- net +5V: now also U1.30 (AVCC), U1.32 (AREF), J1.2 (Pin_2), J3.16 (Pin_16), J3.2 (Pin_2), J3.3 (Pin_3), J4.3 (Pin_3), R2.2
- net GND: now reaches U1.11 (GND), U1.31 (GND)
- net GND: now also C1.2, D1.1 (K), J1.1 (Pin_1), J3.1 (Pin_1), J3.10 (Pin_10), J3.11 (Pin_11), J3.12 (Pin_12), J3.13 (Pin_13), J3.14 (Pin_14), J3.17 (Pin_17), J3.18 (Pin_18), J3.19 (Pin_19), J3.20 (Pin_20), J3.4 (Pin_4), J3.5 (Pin_5), J3.6 (Pin_6), J3.9 (Pin_9), J4.4 (Pin_4)
- net at U1.14 (PD0): now also J4.2 (Pin_2)
- net at U1.15 (PD1): now also J4.1 (Pin_1)
- net at U1.16 (PD2): now also J1.5 (Pin_5)
- net at U1.17 (PD3): now also J1.4 (Pin_4)
- net at U1.2 (PB1): now also J3.15 (Pin_15)
- net at U1.20 (PD6): now also R1.1
- net at U1.5 (PB4): now also J2.1 (Pin_1)
- net at U1.6 (PB5): now also J2.2 (Pin_2), J3.8 (Pin_8)
- net at U1.7 (PB6): now also J2.3 (Pin_3), J3.7 (Pin_7)
- net at U1.8 (PB7): now also J2.4 (Pin_4)
- net at U1.9 (~{RESET}): now also C1.1, R2.1
- new net: D1.2 (A), R1.2
- no-connect marks 0 -> 25

Commit message: actualización de archivos pcb
Parts:
- added SW1: reset, Button_Switch_THT:SW_PUSH_6mm, symbol Switch:SW_Push
- C1: value C_Polarized -> 10uf; footprint (none) -> Capacitor_THT:CP_Radial_D5.0mm_P2.00mm
- D1: value LED -> hearthbeat led; footprint (none) -> LED_THT:LED_D5.0mm
- R1: value R_US -> 330; footprint (none) -> Resistor_THT:R_Axial_DIN0207_L6.3mm_D2.5mm_P7.62mm_Horizontal
- R2: value R_US -> 10k; footprint (none) -> Resistor_THT:R_Axial_DIN0207_L6.3mm_D2.5mm_P7.62mm_Horizontal
Connections:
- net GND: now also SW1.1
- net at C1.1, R2.1, U1.9 (~{RESET}): now also J2.4 (Pin_4), SW1.2
- net at J3.7 (Pin_7), U1.7 (PB6): now also J2.2 (Pin_2); no longer J2.3 (Pin_3)
- net at J3.8 (Pin_8), U1.6 (PB5): now also J2.1 (Pin_1); no longer J2.2 (Pin_2)
- net at U1.5 (PB4): no longer J2.1 (Pin_1)
- net at U1.8 (PB7): now also J2.3 (Pin_3); no longer J2.4 (Pin_4)
- no-connect marks 25 -> 26
Other:
- moved on the sheet: C1, J2, R2
